File: hardware/basic-ecp5-pcb.sch (KiCad schematic (older format))
At the start: 65 parts, among them J1 Conn_01x02, J2 Conn_02x20_Odd_Even, J3 Conn_02x06_Odd_Even, J4 Conn_02x06_Odd_Even, J5 Conn_02x06_Odd_Even, J6 Conn_02x06_Odd_Even, J7 Conn_02x06_Odd_Even, J8 Conn_02x06_Odd_Even, J9 Conn_02x20_Odd_Even, Q1 Q_NMOS_GSD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

Commit message: Initial change setup, deleted stacking connector
Parts:
- removed C10, C22, C4, C5, C6, C8, C9: 100n, Capacitor_SMD:C_0805_2012Metric, symbol Device:C
- removed C11, C15, C26, C7: 10u, Capacitor_SMD:C_0805_2012Metric, symbol Device:C
- removed C12, C13: 4.7u, Capacitor_SMD:C_0805_2012Metric, symbol Device:C
- removed C14: 22u, Capacitor_SMD:C_0805_2012Metric, symbol Device:C
- removed C20, C3: 1u, Capacitor_SMD:C_0805_2012Metric, symbol Device:C
- removed C21: CP, Capacitor_SMD:CP_Elec_5x5.4, symbol Device:CP
- removed D3: LED, LED_SMD:LED_0805_2012Metric, symbol Device:LED
- removed FB1, FB2, FB3: Ferrite_Bead_Small, Inductor_SMD:L_0805_2012Metric, symbol Device:Ferrite_Bead_Small
- removed H1, H2, H3, H4: MountingHole_Pad, MountingHole:MountingHole_3.2mm_M3_Pad, symbol Mechanical:MountingHole_Pad
- removed J1: Conn_01x02, Connector_PinHeader_2.54mm:PinHeader_2x01_P2.54mm_Vertical, symbol Connector_Generic:Conn_01x02
- removed J2: Conn_02x20_Odd_Even, Connector_PinSocket_2.54mm:PinSocket_2x20_P2.54mm_Vertical, symbol Connector_Generic:Conn_02x20_Odd_Even
- removed J5, J6: Conn_02x06_Odd_Even, Connector_PinSocket_2.54mm:PinSocket_2x06_P2.54mm_Horizontal, symbol Connector_Generic:Conn_02x06_Odd_Even
- removed L2, L3: 2.2uH, Inductor_SMD:L_Taiyo-Yuden_NR-40xx, symbol Device:L
- removed R4: 100k, Resistor_SMD:R_0805_2012Metric, symbol Device:R
- removed R5: 120k, Resistor_SMD:R_0805_2012Metric, symbol Device:R
- removed R7: 68k, Resistor_SMD:R_0805_2012Metric, symbol Device:R
- removed R8: 15k, Resistor_SMD:R_0805_2012Metric, symbol Device:R
- removed R9: 200R, Resistor_SMD:R_0805_2012Metric, symbol Device:R
- removed TP1: 3.3v, TestPoint:TestPoint_THTPad_D1.0mm_Drill0.5mm, symbol Connector:TestPoint
- removed TP3: 2.5v, TestPoint:TestPoint_THTPad_D1.0mm_Drill0.5mm, symbol Connector:TestPoint
- removed TP6: 1.1v, TestPoint:TestPoint_THTPad_D1.0mm_Drill0.5mm, symbol Connector:TestPoint
- removed U3, U4: TLV62568DBV, Package_TO_SOT_SMD:SOT-23-5, symbol Regulator_Switching:TLV62568DBV
- removed U5: TLV73325PDBV, Package_TO_SOT_SMD:SOT-23-5, symbol Regulator_Linear:TLV73333PDBV
- U2: symbol Memory_Flash:W25Q128JVS -> basic-ecp5-pcb-rescue:W25Q128JVS-Memory_Flash
- X1: symbol clock:SiT2001B -> basic-ecp5-pcb-rescue:SiT2001B-clock
Connections:
- net labels removed: +1V1, +2V5, 2v5, p3_1, p3_2, p3_3, p3_4, p3_7, p3_8, p4_1, p4_10, p4_2, p4_3, p4_4, p4_7, p4_8, p4_9
- wire segments 73 -> 32
Other:
- note removed: "1.1v @ 1A\n"
- note removed: "2.5v @ 300mA"
- note removed: "3.3v @ 1A\n"
- note removed: "Duplicate port to expose all pins"
- note removed: "Power Supply"
- note removed: "r1"
- note removed: "r2"
- note removed: "vout = 0.6 * (1 + R1/R2)\nvout = 1.1"
- note removed: "vout = 0.6 * (1 + R1/R2)\nvout = 3.32"
