File: hardware/fpga.sch (KiCad schematic (older format))
At the start: 8 parts, among them J10 Conn_02x05_Odd_Even, U1 ECP5U_45_CABGA256

Commit message: Initial change setup, deleted stacking connector
Parts:
- RN1, RN2: symbol Device:R_Pack04_Split -> basic-ecp5-pcb-rescue:R_Pack04_Split-Device
- U1: symbol Lattice_ECP_FPGA:ECP5U_45_CABGA256 -> basic-ecp5-pcb-rescue:ECP5U_45_CABGA256-Lattice_ECP_FPGA
Changed lines of the file:
@@
 EESchema Schematic File Version 4
-EELAYER 30 0
+LIBS:basic-ecp5-pcb-cache
+EELAYER 29 0
 EELAYER END
 $Descr A3 16535 11693
 encoding utf-8
-Sheet 2 2
+Sheet 2 3
 Title "basic ecp5 board"
 Date "2020-07-16"
@@
 $EndDescr
 $Comp
-L Lattice_ECP_FPGA:ECP5U_45_CABGA256 U1
+L basic-ecp5-pcb-rescue:ECP5U_45_CABGA256-Lattice_ECP_FPGA U1
 U 1 1 5F10BE82
 P 10400 7650
@@
 $EndComp
 $Comp
-L Lattice_ECP_FPGA:ECP5U_45_CABGA256 U1
+L basic-ecp5-pcb-rescue:ECP5U_45_CABGA256-Lattice_ECP_FPGA U1
 U 2 1 5F10DDFC
 P 950 2150
@@
 $EndComp
 $Comp
-L Lattice_ECP_FPGA:ECP5U_45_CABGA256 U1
+L basic-ecp5-pcb-rescue:ECP5U_45_CABGA256-Lattice_ECP_FPGA U1
 U 3 1 5F111AF1
 P 3550 2150
@@
 $EndComp
 $Comp
-L Lattice_ECP_FPGA:ECP5U_45_CABGA256 U1
+L basic-ecp5-pcb-rescue:ECP5U_45_CABGA256-Lattice_ECP_FPGA U1
 U 4 1 5F1149C5
 P 6350 2150
@@
 $EndComp
 $Comp
-L Lattice_ECP_FPGA:ECP5U_45_CABGA256 U1
+L basic-ecp5-pcb-rescue:ECP5U_45_CABGA256-Lattice_ECP_FPGA U1
 U 5 1 5F1182AD
 P 9850 2100
@@
 $EndComp
 $Comp
-L Lattice_ECP_FPGA:ECP5U_45_CABGA256 U1
+L basic-ecp5-pcb-rescue:ECP5U_45_CABGA256-Lattice_ECP_FPGA U1
 U 6 1 5F120FEF
 P 13250 2050
@@
 $EndComp
 $Comp
-L Lattice_ECP_FPGA:ECP5U_45_CABGA256 U1
+L basic-ecp5-pcb-rescue:ECP5U_45_CABGA256-Lattice_ECP_FPGA U1
 U 7 1 5F12C303
 P 1450 7400
@@
 $EndComp
 $Comp
-L Lattice_ECP_FPGA:ECP5U_45_CABGA256 U1
+L basic-ecp5-pcb-rescue:ECP5U_45_CABGA256-Lattice_ECP_FPGA U1
 U 9 1 5F14250E
 P 14200 7450
@@
 	6450 7000 6450 6900
 $Comp
-L Device:R_Pack04_Split RN1
+L basic-ecp5-pcb-rescue:R_Pack04_Split-Device RN1
 U 1 1 5F2923DD
 P 5950 9550
+AR Path="/5F2923DD" Ref="RN1"  Part="1"
+AR Path="/5F109712/5F2923DD" Ref="RN1"  Part="1"
 F 0 "RN1" H 6038 9596 50  0001 L CNN
 F 1 "10k" V 5950 9450 50  0000 L CNN
@@
 $EndComp
 $Comp
-L Device:R_Pack04_Split RN1
+L basic-ecp5-pcb-rescue:R_Pack04_Split-Device RN1
 U 2 1 5F2B9F61
 P 6150 7150
+AR Path="/5F2B9F61" Ref="RN1"  Part="2"
+AR Path="/5F109712/5F2B9F61" Ref="RN1"  Part="2"
 F 0 "RN1" H 6238 7196 50  0001 L CNN
 F 1 "10k" V 6150 7100 50  0000 L CNN
@@
 $EndComp
 $Comp
-L Device:R_Pack04_Split RN2
+L basic-ecp5-pcb-rescue:R_Pack04_Split-Device RN2
 U 1 1 5F2BAD04
 P 5750 7150
+AR Path="/5F2BAD04" Ref="RN2"  Part="1"
+AR Path="/5F109712/5F2BAD04" Ref="RN2"  Part="1"
 F 0 "RN2" H 5838 7196 50  0001 L CNN
 F 1 "10k" V 5750 7100 50  0000 L CNN
@@
 $EndComp
 $Comp
-L Device:R_Pack04_Split RN2
+L basic-ecp5-pcb-rescue:R_Pack04_Split-Device RN2
 U 2 1 5F2BBBFC
 P 6250 7150
+AR Path="/5F2BBBFC" Ref="RN2"  Part="2"
+AR Path="/5F109712/5F2BBBFC" Ref="RN2"  Part="2"
 F 0 "RN2" H 5750 7500 50  0001 L CNN
 F 1 "10k" V 6250 7100 50  0000 L CNN
@@
 $EndComp
 $Comp
-L Device:R_Pack04_Split RN2
+L basic-ecp5-pcb-rescue:R_Pack04_Split-Device RN2
 U 3 1 5F2BC5CC
 P 6350 7150
+AR Path="/5F2BC5CC" Ref="RN2"  Part="3"
+AR Path="/5F109712/5F2BC5CC" Ref="RN2"  Part="3"
 F 0 "RN2" H 6600 7500 50  0001 L CNN
 F 1 "10k" V 6350 7100 50  0000 L CNN
@@
 $EndComp
 $Comp
-L Device:R_Pack04_Split RN2
+L basic-ecp5-pcb-rescue:R_Pack04_Split-Device RN2
 U 4 1 5F2BCE12
 P 5850 7150
+AR Path="/5F2BCE12" Ref="RN2"  Part="4"
+AR Path="/5F109712/5F2BCE12" Ref="RN2"  Part="4"
 F 0 "RN2" H 6100 7550 50  0001 L CNN
 F 1 "10k" V 5850 7100 50  0000 L CNN
@@
 $EndComp
 $Comp
-L Device:R_Pack04_Split RN1
+L basic-ecp5-pcb-rescue:R_Pack04_Split-Device RN1
 U 4 1 5F2C115D
 P 6450 7150
+AR Path="/5F2C115D" Ref="RN1"  Part="4"
+AR Path="/5F109712/5F2C115D" Ref="RN1"  Part="4"
 F 0 "RN1" H 6538 7196 50  0001 L CNN
 F 1 "10k" V 6450 7050 50  0000 L CNN
@@
 $EndComp
 $Comp
-L Device:R_Pack04_Split RN1
+L basic-ecp5-pcb-rescue:R_Pack04_Split-Device RN1
 U 3 1 5F2C06DF
 P 6050 9550
+AR Path="/5F2C06DF" Ref="RN1"  Part="3"
+AR Path="/5F109712/5F2C06DF" Ref="RN1"  Part="3"
 F 0 "RN1" H 6138 9596 50  0001 L CNN
 F 1 "10k" V 6050 9450 50  0000 L CNN
@@
 	6250 7450 6600 7450
 $Comp
-L Lattice_ECP_FPGA:ECP5U_45_CABGA256 U1
+L basic-ecp5-pcb-rescue:ECP5U_45_CABGA256-Lattice_ECP_FPGA U1
 U 8 1 5F1343A1
 P 6600 7450
